File: companion/v4/hardware/left/kicad/pcbvr_left.kicad_sch (KiCad schematic)
At the start: 29 parts, among them J1 USB_C_Receptacle_PowerOnly_6P, J2 speaker, J3 TF31-6S-0.5SH_800_, SW1 SW_SPDT, U1 MAX98357AETE_T, U2 BQ24074RGT

Commit message: rev 2 - mcu changes and other various fixes
Other:
- note added: "BT1: 1S LiPo, JST-PH. MUST be a protected cell (built-in PCM: over-discharge, overcharge, overcurrent). Verify red wire = BT1+ before plugging in."
