File: companion/v4/hardware/right/kicad/pcb_right.kicad_sch (KiCad schematic)
At the start: 55 parts, among them J1 TF31-6S-0.5SH_800_, J2 speaker, J3 USB_C_Receptacle_USB2.0_14P, J4 Conn_01x24_MountingPin, SW1 SW_BOOT, SW3 SW_RESET, U2 MAX98357AETE_T, U3 USBLC6-2SC6, U4 ESP32-S3-MINI-1, U5 TLV75528PDBV, U6 TPS63001, U7 TLV75515PDBV

Commit message: Complete right PCB rev 1 layout and BOM
Finish rev 1 layout for the v4 right board, add fabrication outputs
(BOM, positions, netlist, gerbers), shared Master_lib symbols and
footprints, 3D models, and PCB renders.

Co-Authored-By: Claude Opus 5.5 <noreply@anthropic.com>
Parts:
- removed C23: 47uf, Capacitor_SMD:C_0402_1005Metric, symbol Device:C
- removed FB1, FB2: FerriteBead, Inductor_SMD:L_0805_2012Metric_Pad1.05x1.20mm_HandSolder, symbol Device:FerriteBead
- removed L1: 2.2uH, Package_SON:Texas_DRC0010J_ThermalVias, symbol Device:L
- added FB1, FB2: BLM21PG600SN1D, Master_lib:BLM21AG102BH1J, symbol Lib_Solar_panels:BLM21PG600SN1D
- added JP3: SolderJumper_2_Open, Jumper:SolderJumper-2_P1.3mm_Open_RoundedPad1.0x1.5mm, symbol Jumper:SolderJumper_2_Open
- added L1: 2.2uH, Master_lib:INDC2520X120N, symbol Master_lib:DFE252012F-2R2M=P2
- added TP4, TP5, TP6: GND, TestPoint:TestPoint_Pad_D1.5mm, symbol Connector:TestPoint
- C1, C2: value 220PF -> 220pF; JLCPCB_Part# (none) -> C107145; Manufacturer_Part_Number (none) -> CC0805KRX7R9BB221
- C10: value 1u -> 1uF; JLCPCB_Part# (none) -> C52923; Manufacturer_Part_Number (none) -> CL05A105KA5NQNC
- C11, C12, C14, C15, C17, C19, C21: value 1uf -> 1uF; JLCPCB_Part# (none) -> C52923; Manufacturer_Part_Number (none) -> CL05A105KA5NQNC
- C13, C16: value 100n -> 0.1uF; JLCPCB_Part# (none) -> C1525; Manufacturer_Part_Number (none) -> CL05B104KO5NNNC
- C18, C20, C22: value 100nf -> 0.1uF; JLCPCB_Part# (none) -> C1525; Manufacturer_Part_Number (none) -> CL05B104KO5NNNC
- C24, C26, C27, C8: value 10uf -> 10uF; JLCPCB_Part# (none) -> C315248; Manufacturer_Part_Number (none) -> CL05A106MP5NUNC
- C25, C28, C9: value 0.1uf -> 0.1uF; JLCPCB_Part# (none) -> C1525; Manufacturer_Part_Number (none) -> CL05B104KO5NNNC
- C3: value 0.1UF -> 0.1uF; JLCPCB_Part# (none) -> C49678; Manufacturer_Part_Number (none) -> CC0805KRX7R9BB104
- C4: value 10UF -> 10uF; JLCPCB_Part# (none) -> C15850; Manufacturer_Part_Number (none) -> CL21A106KAYNNNE
- J1: footprint HRS_TF31-6S-0.5SH_800_:HRS_TF31-6S-0.5SH_800_ -> Master_lib:HRS_TF31-6S-0.5SH_800_; JLCPCB_Part# (none) -> C3195341; Manufacturer_Part_Number (none) -> TF31-6S-0.5SH(800)
- J2: now not fitted; now left out of the parts list
- J3: footprint Connector_USB:USB_C_Receptacle_HRO_TYPE-C-31-M-12 -> Master_lib:USB_C_Receptacle_HRO_TYPE-C-31-M-12; JLCPCB_Part# (none) -> C165948; Manufacturer_Part_Number (none) -> TYPE-C-31-M-12
- J4: JLCPCB_Part# (none) -> C202112; Manufacturer_Part_Number (none) -> FH12-24S-0.5SH(55)
- R1, R2: value 100k -> 100K; JLCPCB_Part# (none) -> C149504; Manufacturer_Part_Number (none) -> 0805W8F1003T5E
- R10, R9: value 10k -> 10K; JLCPCB_Part# (none) -> C17414; Manufacturer_Part_Number (none) -> 0805W8F1002T5E
- R11, R4: value 10kΩ -> 10K; JLCPCB_Part# (none) -> C25744; Manufacturer_Part_Number (none) -> 0402WGF1002TCE
- R3: value 100 -> 100R; JLCPCB_Part# (none) -> C17408; Manufacturer_Part_Number (none) -> 0805W8F1000T5E
- R5, R6: value 5.1kΩ -> 5.1K; JLCPCB_Part# (none) -> C25905; Manufacturer_Part_Number (none) -> 0402WGF5101TCE
- R7, R8: value 4.7k -> 4.7K; JLCPCB_Part# (none) -> C17673; Manufacturer_Part_Number (none) -> 0805W8F4701T5E
- SW1, SW3: footprint Button_Switch_THT:SW_PUSH_6mm_H5mm -> Button_Switch_SMD:SW_SPST_PTS810; JLCPCB_Part# (none) -> C221895; Manufacturer_Part_Number (none) -> PTS810SJG250SMTRLFS
- TP1: footprint Package_TO_SOT_SMD:SOT-23-5 -> TestPoint:TestPoint_Pad_D1.5mm; now left out of the parts list
- TP2, TP3: now left out of the parts list
- U2: footprint MAX98357A:QFN50P300X300X80-17N -> Master_lib:QFN50P300X300X80-17N; Description_1 Tiny, Low-Cost, PCM Class D Amplifier with Class AB Perform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 -> (none); JLCPCB_Part# (none) -> C910544; Manufacturer_Part_Number (none) -> MAX98357AETE+T
- U3: JLCPCB_Part# (none) -> C7519; Manufacturer_Part_Number (none) -> USBLC6-2SC6
- U4: footprint RF_Module:ESP32-S2-MINI-1 -> Master_lib:ESP32-S2-MINI-1; JLCPCB_Part# (none) -> C3013941; Manufacturer_Part_Number (none) -> ESP32-S3-MINI-1-N4R2
- U5: JLCPCB_Part# (none) -> C2868951; Manufacturer_Part_Number (none) -> TLV75528PDBVR
- U6: footprint Package_SON:Texas_DRC0010J_ThermalVias -> Master_lib:Texas_DRC0010J_ThermalVias; JLCPCB_Part# (none) -> C28060; Manufacturer_Part_Number (none) -> TPS63001DRCR
- U7: JLCPCB_Part# (none) -> C2867152; Manufacturer_Part_Number (none) -> TLV75515PDBVR
Connections:
- net +3.3V: now also TP4.1
- net +5V: now also JP3.2 (B), TP5.1
- net GND: now also TP6.1
- net USB_DN: now also U3.1 (I/O1), U3.6 (I/O1); no longer U3.3 (I/O2), U3.4 (I/O2)
- net USB_DP: now also U3.3 (I/O2), U3.4 (I/O2); no longer U3.1 (I/O1), U3.6 (I/O1)
- net at U2.10 (OUTN): now also FB1.1
- net at C2.2, J2.2 (Pin_2): now also FB1.2
- net at U2.9 (OUTP): now also FB2.1
- net at C1.1, J2.1 (Pin_1): now also FB2.2
- net at J3.A4 (VBUS), J3.A9 (VBUS), J3.B4 (VBUS)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: now also JP3.1 (A)
- net at U6.2 (L2): now also L1.1
- net at U6.4 (L1): now also L1.2
- no-connect marks 20 -> 19
Other:
- moved on the sheet: C26, C27, TP3, U6
